File: PCB/keyboard.kicad_pcb (KiCad board)
At the start: 2 copper layers, 285.5 x 95 mm, 136 parts, among them J1 USB_C_Receptacle, U1 ATmega32U4-M

Commit message: first routing
Parts:
- removed the REF** at (130.8, 85.6)
- removed the REF** at (128.2, 47.0)
- removed the REF** at (259.4, 66.5)
- removed the REF** at (21.3, 66.5)
- removed the REF** at (264.2, 47.5)
- added C1: 1uF, Capacitor_SMD:C_0603_1608Metric_Pad1.08x0.95mm_HandSolder, B.Cu at (331.0, 223.6)
- added C2: 0.1uF, Capacitor_SMD:C_0603_1608Metric_Pad1.08x0.95mm_HandSolder, B.Cu at (335.4, 231.1)
- added C3: 10uF, Capacitor_SMD:C_0603_1608Metric_Pad1.08x0.95mm_HandSolder, B.Cu at (323.2, 230.2)
- added C4: 0.1uF, Capacitor_SMD:C_0603_1608Metric_Pad1.08x0.95mm_HandSolder, B.Cu at (322.5, 236.5)
- added C5: 0.1uF, Capacitor_SMD:C_0603_1608Metric_Pad1.08x0.95mm_HandSolder, B.Cu at (331.7, 240.5)
- added C6: 22pF, Capacitor_SMD:C_0603_1608Metric_Pad1.08x0.95mm_HandSolder, B.Cu at (338.5, 239.3)
- added C7: 22pF, Capacitor_SMD:C_0603_1608Metric_Pad1.08x0.95mm_HandSolder, B.Cu at (339.7, 230.2)
- added C8: 0.1uF, Capacitor_SMD:C_0603_1608Metric_Pad1.08x0.95mm_HandSolder, B.Cu at (332.6, 223.6)
- added C9: 0.1uF, Capacitor_SMD:C_0603_1608Metric_Pad1.08x0.95mm_HandSolder, B.Cu at (324.7, 226.3)
- added F1: 500mA, Fuse:Fuse_1206_3216Metric_Pad1.42x1.75mm_HandSolder, B.Cu at (308.5, 168.8)
- added R1: 22, Resistor_SMD:R_0603_1608Metric_Pad0.98x0.95mm_HandSolder, B.Cu at (327.6, 226.3)
- added R2: 22, Resistor_SMD:R_0603_1608Metric_Pad0.98x0.95mm_HandSolder, B.Cu at (326.1, 226.3)
- added R3: 5.1k, Resistor_SMD:R_0603_1608Metric_Pad0.98x0.95mm_HandSolder, B.Cu at (300.9, 160.0)
- added R4: 5.1k, Resistor_SMD:R_0603_1608Metric_Pad0.98x0.95mm_HandSolder, B.Cu at (305.5, 161.8)
- added R5: 10k, Resistor_SMD:R_0603_1608Metric_Pad0.98x0.95mm_HandSolder, B.Cu at (324.0, 238.8)
- added R6: 10k, Resistor_SMD:R_0603_1608Metric_Pad0.98x0.95mm_HandSolder, B.Cu at (326.9, 217.3)
- added REF**: MountingHole_7mm_2.5mm_M2_Pad, custom_mounting_hole:MountingHole_7mm_2.5mm_M2_Pad, F.Cu at (298.4, 197.1)
- added REF**: Stabilizer_Cherry_MX_2.00u, keyboard_stabilizer:Stabilizer_Cherry_MX_2.00u, F.Cu at (434.2, 197.5)
- added REF**: Stabilizer_Cherry_MX_2.00u, keyboard_stabilizer:Stabilizer_Cherry_MX_2.00u, F.Cu at (191.3, 216.6)
- added REF**: Stabilizer_Cherry_MX_2.00u, keyboard_stabilizer:Stabilizer_Cherry_MX_2.00u, F.Cu at (429.4, 216.6)
- added REF**: Stabilizer_Cherry_MX_6.25u, keyboard_stabilizer:Stabilizer_Cherry_MX_6.25u, F.Cu at (300.8, 235.6)
- added SW1: SW_Push, Button_Switch_SMD:SW_Push_1P1T_XKB_TS-1187A, B.Cu at (199.2, 198.2)
- added Y1: 16MHz, Crystal:Crystal_SMD_3225-4Pin_3.2x2.5mm_HandSoldering, B.Cu at (338.5, 235.0)
- D_0, D_1, D_10, D_11, D_12, D_13, D_14, D_15, D_16, D_17, D_18, D_19, D_2, D_20, D_21, D_22, D_23, D_24, D_25, D_26, D_27, D_28, D_29, D_3, D_30, D_31, D_32, D_33, D_34, D_35, D_36, D_37, D_38, D_39, D_4, D_40, D_41, D_42, D_43, D_44, D_45, D_46, D_47, D_48, D_49, D_5, D_50, D_51, D_52, D_53, D_54, D_55, D_56, D_57, D_58, D_59, D_6, D_60, D_61, D_7, D_8, D_9: footprint Diode_SMD:D_SOD-123 -> custom_components:D_SOD-123_vertical
- J1: footprint Connector_USB:USB_C_Receptacle_G-Switch_GT-USB-7010ASV -> custom_components:USB_C_Receptacle_G-Switch_GT-USB-7010ASV_custom
- moved U1 230.2 mm to (328.6, 233.6), turned to -90 degrees
- moved D_7 229.6 mm to (321.0, 164.5)
- moved D_14 226.9 mm to (448.8, 164.5)
- moved D_28 226.9 mm to (444.0, 183.5)
- moved D_53 226.9 mm to (432.0, 221.8)
- moved K_21 226.7 mm to (303.2, 178.4)
- moved K_26 226.7 mm to (398.5, 178.4)
- moved K_36 226.7 mm to (327.0, 197.5)
- moved K_46 226.7 mm to (279.4, 216.6)
- moved K_51 226.7 mm to (374.7, 216.6)
- moved K_9 226.7 mm to (350.9, 159.4)
- moved D_10 226.7 mm to (372.5, 164.5)
- moved D_11 226.7 mm to (391.5, 164.5)
- moved D_12 226.7 mm to (410.5, 164.5)
- moved D_13 226.7 mm to (429.5, 164.5)
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Connections:
- J1 pad A4: VCC -> Net-(F1-Pad2)
- J1 pad A5: unconnected-(J1-CC1-PadA5) -> Net-(J1-CC1)
- J1 pad A6: unconnected-(J1-D+-PadA6) -> D+
- J1 pad A7: unconnected-(J1-D--PadA7) -> D-
- J1 pad A9: VCC -> Net-(F1-Pad2)
- J1 pad B4: VCC -> Net-(F1-Pad2)
- J1 pad B5: unconnected-(J1-CC2-PadB5) -> Net-(J1-CC2)
- J1 pad B6: unconnected-(J1-D+-PadB6) -> D+
- J1 pad B7: unconnected-(J1-D--PadB7) -> D-
- J1 pad B9: VCC -> Net-(F1-Pad2)
- U1 pad 10: unconnected-(U1-PB2-Pad10) -> col8
- U1 pad 11: unconnected-(U1-PB3-Pad11) -> col9
- U1 pad 13: unconnected-(U1-~{RESET}-Pad13) -> Net-(U1-~{RESET})
- U1 pad 14: Net-(U1-VCC-Pad14) -> VCC
- U1 pad 15: Net-(U1-GND-Pad15) -> GND
- U1 pad 16: unconnected-(U1-XTAL2-Pad16) -> Net-(U1-XTAL2)
- U1 pad 17: unconnected-(U1-XTAL1-Pad17) -> Net-(U1-XTAL1)
- U1 pad 18: unconnected-(U1-PD0-Pad18) -> col10
- U1 pad 19: unconnected-(U1-PD1-Pad19) -> col12
- U1 pad 2: unconnected-(U1-UVCC-Pad2) -> VCC
- U1 pad 20: unconnected-(U1-PD2-Pad20) -> col11
- U1 pad 21: unconnected-(U1-PD3-Pad21) -> col14
- U1 pad 22: unconnected-(U1-PD5-Pad22) -> col13
- U1 pad 23: Net-(U1-GND-Pad15) -> GND
- U1 pad 24: Net-(U1-AVCC-Pad24) -> VCC
- U1 pad 26: unconnected-(U1-PD6-Pad26) -> col6
- U1 pad 27: unconnected-(U1-PD7-Pad27) -> col0
- U1 pad 28: unconnected-(U1-PB4-Pad28) -> col1
- U1 pad 29: unconnected-(U1-PB5-Pad29) -> col2
- U1 pad 3: unconnected-(U1-D--Pad3) -> Net-(U1-D-)
- U1 pad 30: unconnected-(U1-PB6-Pad30) -> col3
- U1 pad 31: unconnected-(U1-PC6-Pad31) -> col4
- U1 pad 32: unconnected-(U1-PC7-Pad32) -> col5
- U1 pad 33: unconnected-(U1-~{HWB}/PE2-Pad33) -> Net-(U1-~{HWB}/PE2)
- U1 pad 34: Net-(U1-VCC-Pad14) -> VCC
- U1 pad 35: Net-(U1-GND-Pad15) -> GND
- U1 pad 36: unconnected-(U1-PF7-Pad36) -> row4
- U1 pad 37: unconnected-(U1-PF6-Pad37) -> row3
- U1 pad 38: unconnected-(U1-PF5-Pad38) -> row2
- U1 pad 39: unconnected-(U1-PF4-Pad39) -> row1
- U1 pad 4: unconnected-(U1-D+-Pad4) -> Net-(U1-D+)
- U1 pad 40: unconnected-(U1-PF1-Pad40) -> row0
- U1 pad 41: unconnected-(U1-PF0-Pad41) -> col7
- U1 pad 43: Net-(U1-GND-Pad15) -> GND
- U1 pad 44: Net-(U1-AVCC-Pad24) -> VCC
- U1 pad 45: Net-(U1-GND-Pad15) -> GND
- U1 pad 5: unconnected-(U1-UGND-Pad5) -> GND
- U1 pad 6: unconnected-(U1-UCAP-Pad6) -> Net-(U1-UCAP)
- U1 pad 7: unconnected-(U1-VBUS-Pad7) -> VCC
Routing:
- net row0: track 0.00 -> 353.4 mm, vias 0 -> 2
- net row1: track 0.00 -> 328.5 mm, vias 0 -> 2
- net row2: track 0.00 -> 295.3 mm, vias 0 -> 2
- net row4: track 0.00 -> 282.7 mm, vias 0 -> 2
- net row3: track 0.00 -> 272.1 mm
- net col0: track 0.00 -> 248.4 mm
- net col1: track 0.00 -> 229.3 mm, vias 0 -> 1
- net col2: track 0.00 -> 199.7 mm, vias 0 -> 1
- net col3: track 0.00 -> 196.1 mm, vias 0 -> 1
- net Net-(U1-~{RESET}): track 0.00 -> 168.7 mm, vias 0 -> 3
- net col11: track 0.00 -> 158.7 mm, vias 0 -> 1
- net col12: track 0.00 -> 154.8 mm, vias 0 -> 1
- net col4: track 0.00 -> 153.9 mm, vias 0 -> 1
- net col10: track 0.00 -> 138.9 mm, vias 0 -> 1
- net col5: track 0.00 -> 137.6 mm, vias 0 -> 1
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