File: PCB/v0.2/keyboard.kicad_pcb (KiCad board)
At the start: 2 copper layers, 285.5 x 95 mm, 155 parts, among them J1 USB_C_Receptacle, SW1 SW_Push, U1 ATmega32U4-M, Y1 16MHz

Commit message: dfasdasfawef
Parts:
- removed C1: 1uF, Capacitor_SMD:C_0603_1608Metric_Pad1.08x0.95mm_HandSolder
- removed C10, C2, C4, C5, C8, C9: 0.1uF, Capacitor_SMD:C_0603_1608Metric_Pad1.08x0.95mm_HandSolder
- removed C3: 10uF, Capacitor_SMD:C_0603_1608Metric_Pad1.08x0.95mm_HandSolder
- removed C6, C7: 22pF, Capacitor_SMD:C_0603_1608Metric_Pad1.08x0.95mm_HandSolder
- removed R5, R6: 10k, Resistor_SMD:R_0603_1608Metric_Pad0.98x0.95mm_HandSolder
- removed REF** (x3): Stabilizer_Cherry_MX_2.00u, keyboard_stabilizer:Stabilizer_Cherry_MX_2.00u
- removed REF** (x2): MountingHole_7mmx2.5mm_M2_Pad, custom_mounting_hole:MountingHole_7mmx2.5mm_M2_Pad
- removed REF**: Stabilizer_Cherry_MX_6.25u, keyboard_stabilizer:Stabilizer_Cherry_MX_6.25u
- removed REF**: MountingHole_7mm_2.5mm_M2_Pad, custom_mounting_hole:MountingHole_7mm_2.5mm_M2_Pad
- removed REF** (x2): MountingHole_5mmx2.5mm_M2_Pad, custom_mounting_hole:MountingHole_5mmx2.5mm_M2_Pad
- removed REF**: MountingHole_2.5mm_M2_Pad, custom_mounting_hole:MountingHole_2.5mm_M2_Pad
- removed SW1: SW_Push, Button_Switch_SMD:SW_Push_1P1T_XKB_TS-1187A
- removed Y1: 16MHz, Crystal:Crystal_SMD_3225-4Pin_3.2x2.5mm_HandSoldering
- added BOOT1: SW_SPST, Button_Switch_SMD:SW_SPST_TL3342, B.Cu at (231.8, 192.8)
- added C11: 100nF, Capacitor_SMD:C_0402_1005Metric, B.Cu at (245.8, 188.2)
- added C12: 10uF, Capacitor_SMD:C_0603_1608Metric, B.Cu at (248.6, 190.1)
- added C13: 100nF, Capacitor_SMD:C_0402_1005Metric, B.Cu at (263.1, 199.0)
- added C14: 1uF, Capacitor_SMD:C_0402_1005Metric, B.Cu at (250.7, 182.5)
- added C15: 100nF, Capacitor_SMD:C_0402_1005Metric, B.Cu at (252.5, 195.6)
- added C16: 100nF, Capacitor_SMD:C_0402_1005Metric, B.Cu at (255.4, 198.4)
- added C17: 1uF, Capacitor_SMD:C_0402_1005Metric, B.Cu at (250.7, 187.5)
- added C18: 100nF, Capacitor_SMD:C_0402_1005Metric, B.Cu at (267.0, 188.1)
- added C19: 100nF, Capacitor_SMD:C_0402_1005Metric, B.Cu at (255.4, 183.5)
- added C20: 100nF, Capacitor_SMD:C_0402_1005Metric, B.Cu at (253.9, 196.9)
- added D_62: D, custom_components:D_SOD-123_vertical, B.Cu at (176.7, 178.6)
- added D_63: D, custom_components:D_SOD-123_vertical, B.Cu at (431.4, 178.6)
- added D_64: D, custom_components:D_SOD-123_vertical, B.Cu at (423.6, 159.2)
- added F2: 500mA, Fuse:Fuse_1206_3216Metric, B.Cu at (287.6, 121.0)
- added F4: 500mA, Fuse:Fuse_1206_3216Metric, B.Cu at (181.0, 151.9)
- added H10: MountingHole_Pad, custom_mounting_hole:MountingHole_5mmx2.5mm_M2_Pad, B.Cu at (343.5, 193.2)
- added H11: MountingHole_Pad, custom_mounting_hole:MountingHole_5mmx2.5mm_M2_Pad, B.Cu at (413.1, 135.9)
- added H12: MountingHole_Pad, custom_mounting_hole:MountingHole_2.5mm_M2_Pad, B.Cu at (178.2, 135.9)
- added H7: MountingHole_Pad, custom_mounting_hole:MountingHole_7mmx2.5mm_M2_Pad, B.Cu at (155.2, 164.5)
- added H8: MountingHole_Pad, custom_mounting_hole:MountingHole_7mmx2.5mm_M2_Pad, B.Cu at (436.6, 164.3)
- added H9: MountingHole_Pad, custom_mounting_hole:MountingHole_7mm_2.5mm_M2_Pad, B.Cu at (281.2, 155.0)
- added J2: USB_C_Receptacle_USB2.0_16P, custom_components:USB_C_Receptacle_G-Switch_GT-USB-7010ASV_custom, B.Cu at (295.5, 110.7)
- added J4: Conn_01x04_MountingPin, Connector_Molex:Molex_Pico-EZmate_78171-0004_1x04-1MP_P1.20mm_Vertical, B.Cu at (177.5, 146.1)
- added J8: Conn_01x04_Socket, Connector_PinHeader_2.54mm:PinHeader_1x04_P2.54mm_Vertical, B.Cu at (182.3, 148.7)
- added K_62: KEYSW, keyboard_switches:SW_Cherry_MX_PCB, F.Cu at (295.5, 193.4)
- added K_63: KEYSW, keyboard_switches:SW_Cherry_MX_PCB, F.Cu at (276.4, 193.4)
- added K_64: KEYSW, keyboard_switches:SW_Cherry_MX_PCB, F.Cu at (166.9, 193.4)
- added K_65: KEYSW, keyboard_switches:SW_Cherry_MX_PCB, F.Cu at (190.8, 193.4)
- added K_66: KEYSW, keyboard_switches:SW_Cherry_MX_PCB, F.Cu at (214.5, 193.4)
- added K_67: KEYSW, keyboard_switches:SW_Cherry_MX_PCB, F.Cu at (357.4, 193.4)
- added K_68: KEYSW, keyboard_switches:SW_Cherry_MX_PCB, F.Cu at (195.5, 193.4)
- added K_69: KEYSW, keyboard_switches:SW_Cherry_MX_PCB, F.Cu at (376.5, 193.4)
- added K_70: KEYSW, keyboard_switches:SW_Cherry_MX_PCB, F.Cu at (381.2, 193.4)
- added K_71: KEYSW, keyboard_switches:SW_Cherry_MX_PCB, F.Cu at (400.3, 193.4)
- added K_72: KEYSW, keyboard_switches:SW_Cherry_MX_PCB, F.Cu at (424.1, 193.4)
- added K_73: KEYSW, keyboard_switches:SW_Cherry_MX_PCB_1.25u, F.Cu at (164.5, 174.3)
- added K_74: KEYSW, keyboard_switches:SW_Cherry_MX_PCB_1.00u, F.Cu at (185.9, 174.3)
- added K_75: KEYSW, keyboard_switches:SW_Cherry_MX_PCB_1.00u, F.Cu at (395.5, 174.3)
- added K_76: KEYSW, keyboard_switches:SW_Cherry_MX_PCB_1.75u, F.Cu at (402.6, 174.3)
- added K_77: KEYSW, keyboard_switches:SW_Cherry_MX_PCB_1.00u, F.Cu at (428.9, 174.3)
- added K_78: KEYSW, keyboard_switches:SW_Cherry_MX_PCB_1.75u, F.Cu at (421.7, 174.3)
- added K_79: KEYSW, keyboard_switches:SW_Cherry_MX_PCB_1.00u, F.Cu at (405.1, 155.3)
- added K_80: KEYSW, keyboard_switches:SW_Cherry_MX_PCB_ISOEnter, F.Cu at (426.5, 145.8)
- added R10: 5.1k, Resistor_SMD:R_0402_1005Metric, B.Cu at (266.0, 197.6)
- added R9: 5.1k, Resistor_SMD:R_0402_1005Metric, B.Cu at (264.6, 197.6)
- added RST1: SW_SPST, Button_Switch_SMD:SW_SPST_TL3342, B.Cu at (239.6, 192.8)
- added S1: MX_stab, keyboard_stabilizer:Stabilizer_Cherry_MX_2.00u, F.Cu at (174.1, 174.3)
- added S2: MX_stab, keyboard_stabilizer:Stabilizer_Cherry_MX_2.00u, F.Cu at (416.9, 155.3)
- added S3: MX_stab, keyboard_stabilizer:Stabilizer_Cherry_MX_2.00u, F.Cu at (412.2, 174.3)
- added S4: MX_stab, keyboard_stabilizer:Stabilizer_Cherry_MX_6.25u, F.Cu at (283.6, 193.4)
- added S5: MX_stab, keyboard_stabilizer:Stabilizer_Cherry_MX_7.00u, F.Cu at (295.5, 193.4)
- added S6: MX_stab, keyboard_stabilizer:Stabilizer_Cherry_MX_single, F.Cu at (219.3, 193.4)
- added S7: MX_stab, keyboard_stabilizer:Stabilizer_Cherry_MX_2.00u, F.Cu at (426.5, 145.8)
- added U3: STM32F072C8Tx, Package_QFP:LQFP-48_7x7mm_P0.5mm, B.Cu at (259.3, 191.2)
- added U4: PRTR5V0U2X, Package_TO_SOT_SMD:SOT-143, B.Cu at (245.7, 185.8)
- F1: footprint Fuse:Fuse_1206_3216Metric_Pad1.42x1.75mm_HandSolder -> Fuse:Fuse_1206_3216Metric
- J1: value USB_C_Receptacle -> USB_C_Receptacle_USB2.0_16P
- R1, R2: value 22 -> 5.1k
- U1: value ATmega32U4-M -> XC6206PxxxMR; footprint custom_components:QFN-44-1EP_7x7mm_P0.5mm_EP5.2x5.2mm -> Package_TO_SOT_SMD:SOT-23-3
- moved R1 195.1 mm to (170.0, 119.5), turned to -90 degrees
- moved R2 191.1 mm to (172.9, 119.5), turned to 90 degrees
- moved F1 153.5 mm to (167.4, 122.7), turned to 0 degrees
- moved J1 147.6 mm to (171.2, 110.9)
- moved U1 90.6 mm to (250.7, 185.0), turned to 180 degrees
- moved D_60 54.7 mm to (408.3, 187.9), turned to -90 degrees
- moved D_61 54.7 mm to (432.1, 187.9), turned to -90 degrees
- moved D_59 54.2 mm to (386.7, 187.9), turned to -90 degrees
- moved D_58 54.1 mm to (363.0, 187.9), turned to -90 degrees
- moved D_54 54.1 mm to (173.1, 187.9), turned to -90 degrees
- moved D_55 53.3 mm to (201.5, 187.9), turned to -90 degrees
- moved D_56 53.0 mm to (222.7, 188.6)
- moved D_57 52.9 mm to (301.3, 187.9), turned to -90 degrees
- moved D_41 51.3 mm to (409.1, 159.2)
- moved D_28 49.8 mm to (418.6, 140.7)
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Connections:
- F1 pad 1: VCC -> Net-(F1-Pad1)
- F1 pad 2: Net-(F1-Pad2) -> +5V
- J1 pad A4: Net-(F1-Pad2) -> Net-(F1-Pad1)
- J1 pad A9: Net-(F1-Pad2) -> Net-(F1-Pad1)
- J1 pad B4: Net-(F1-Pad2) -> Net-(F1-Pad1)
- J1 pad B9: Net-(F1-Pad2) -> Net-(F1-Pad1)
- K_41 pad 1: col13 -> col14
- K_41 pad 2: Net-(D_41-A) -> Net-(D_64-A)
- K_42 pad 1: col1 -> col0
- K_42 pad 2: Net-(D_42-A) -> Net-(D_62-A)
- R1 pad 1: D+ -> Net-(J1-CC1)
- R1 pad 2: Net-(U1-D+) -> GND
- R2 pad 1: D- -> GND
- R2 pad 2: Net-(U1-D-) -> Net-(J1-CC2)
- R3 pad 1: Net-(J1-CC1) -> Net-(J2-CC1)
- R4 pad 2: Net-(J1-CC2) -> Net-(J2-CC2)
- U1 pad 1: unconnected-(U1-PE6-Pad1) -> GND
- U1 pad 2: VCC -> +3V3
- U1 pad 3: Net-(U1-D-) -> +5V
Routing:
- net +5V: track 0.00 -> 264.7 mm, vias 0 -> 6
- net D+: track 102.9 -> 320.9 mm, vias 2 -> 10
- net D-: track 102.0 -> 319.7 mm, vias 3 -> 11
- net Net-(U1-~{RESET}): track 146.8 -> 0.00 mm, vias 1 -> 0
- net col10: track 96.4 -> 193.5 mm, vias 0 -> 1
- net VCC: track 94.4 -> 0.00 mm, vias 2 -> 0
- net +3V3: track 0.00 -> 78.2 mm
- net col8: track 67.2 -> 137.6 mm, vias 0 -> 1
- net col14: track 201.8 -> 263.6 mm
- net col1: track 219.6 -> 159.4 mm
- net col11: track 155.4 -> 214.3 mm, vias 1 -> 3
- net col13: track 191.2 -> 246.8 mm
- net col7: track 93.1 -> 144.9 mm
- net col9: track 99.6 -> 150.7 mm
- net col0: track 238.4 -> 187.2 mm, vias 0 -> 1
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Other:
- board size 285.5 x 95 mm -> 284.7 x 94.2 mm
- board text added: "v-score on left side"
- board text added: "v-score on right side"
