File: PCB/v0.2/keyboard.kicad_sch (KiCad schematic)
At the start: 145 parts, among them J1 USB_C_Receptacle, SW1 SW_Push, U1 ATmega32U4-M, Y1 16MHz

Commit message: dfasdasfawef
Parts:
- removed C1: 1uF, Capacitor_SMD:C_0603_1608Metric_Pad1.08x0.95mm_HandSolder, symbol Device:C
- removed C10, C2, C4, C5, C8, C9: 0.1uF, Capacitor_SMD:C_0603_1608Metric_Pad1.08x0.95mm_HandSolder, symbol Device:C
- removed C3: 10uF, Capacitor_SMD:C_0603_1608Metric_Pad1.08x0.95mm_HandSolder, symbol Device:C
- removed C6, C7: 22pF, Capacitor_SMD:C_0603_1608Metric_Pad1.08x0.95mm_HandSolder, symbol Device:C
- removed J1: USB_C_Receptacle, custom_components:USB_C_Receptacle_G-Switch_GT-USB-7010ASV_custom, symbol Connector:USB_C_Receptacle
- removed R5, R6: 10k, Resistor_SMD:R_0603_1608Metric_Pad0.98x0.95mm_HandSolder, symbol Device:R
- removed SW1: SW_Push, Button_Switch_SMD:SW_Push_1P1T_XKB_TS-1187A, symbol Switch:SW_Push
- removed U1: ATmega32U4-M, Package_DFN_QFN:QFN-44-1EP_7x7mm_P0.5mm_EP5.2x5.2mm, symbol MCU_Microchip_ATmega:ATmega32U4-M
- removed Y1: 16MHz, Crystal:Crystal_SMD_3225-4Pin_3.2x2.5mm_HandSoldering, symbol Device:Crystal_GND24_Small
- added BOOT1, RST1: SW_SPST, Button_Switch_SMD:SW_SPST_TL3342, symbol Switch:SW_SPST
- added C11, C13, C15, C16, C18, C19: 100nF, Capacitor_SMD:C_0402_1005Metric, symbol Device:C
- added C12: 10uF, Capacitor_SMD:C_0603_1608Metric, symbol Device:C
- added C14, C17: 1uF, Capacitor_SMD:C_0402_1005Metric, symbol Device:C
- added C20: 100nF, Capacitor_SMD:C_0402_1005Metric, symbol Device:C_Small
- added D_62, D_63, D_64: D, custom_components:D_SOD-123_vertical, symbol Device:D_Small
- added F2, F4: 500mA, Fuse:Fuse_1206_3216Metric, symbol Device:Polyfuse
- added H10, H11: MountingHole_Pad, custom_mounting_hole:MountingHole_5mmx2.5mm_M2_Pad, symbol Mechanical:MountingHole_Pad
- added H12: MountingHole_Pad, custom_mounting_hole:MountingHole_2.5mm_M2_Pad, symbol Mechanical:MountingHole_Pad
- added H7, H8: MountingHole_Pad, custom_mounting_hole:MountingHole_7mmx2.5mm_M2_Pad, symbol Mechanical:MountingHole_Pad
- added H9: MountingHole_Pad, custom_mounting_hole:MountingHole_7mm_2.5mm_M2_Pad, symbol Mechanical:MountingHole_Pad
- added J1, J2: USB_C_Receptacle_USB2.0_16P, custom_components:USB_C_Receptacle_G-Switch_GT-USB-7010ASV_custom, symbol Connector:USB_C_Receptacle_USB2.0_16P
- added J4: Conn_01x04_MountingPin, Connector_Molex:Molex_Pico-EZmate_78171-0004_1x04-1MP_P1.20mm_Vertical, symbol Connector_Generic_MountingPin:Conn_01x04_MountingPin
- added J8: Conn_01x04_Socket, Connector_PinHeader_2.54mm:PinHeader_1x04_P2.54mm_Vertical, symbol Connector:Conn_01x04_Socket
- added K_62, K_63, K_64, K_65, K_66, K_67, K_68, K_69, K_70, K_71, K_72: KEYSW, keyboard_switches:SW_Cherry_MX_PCB, symbol MX_Alps_Hybrid:MX-NoLED
- added K_73: KEYSW, keyboard_switches:SW_Cherry_MX_PCB_1.25u, symbol MX_Alps_Hybrid:MX-NoLED
- added K_74, K_75, K_77, K_79: KEYSW, keyboard_switches:SW_Cherry_MX_PCB_1.00u, symbol MX_Alps_Hybrid:MX-NoLED
- added K_76, K_78: KEYSW, keyboard_switches:SW_Cherry_MX_PCB_1.75u, symbol MX_Alps_Hybrid:MX-NoLED
- added K_80: KEYSW, keyboard_switches:SW_Cherry_MX_PCB_ISOEnter, symbol MX_Alps_Hybrid:MX-NoLED
- added R10, R9: 5.1k, Resistor_SMD:R_0402_1005Metric, symbol Device:R
- added S1, S2, S3, S7: MX_stab, keyboard_stabilizer:Stabilizer_Cherry_MX_2.00u, symbol marbastlib-mx:MX_stab
- added S4: MX_stab, keyboard_stabilizer:Stabilizer_Cherry_MX_6.25u, symbol marbastlib-mx:MX_stab
- added S5: MX_stab, keyboard_stabilizer:Stabilizer_Cherry_MX_7.00u, symbol marbastlib-mx:MX_stab
- added S6: MX_stab, keyboard_stabilizer:Stabilizer_Cherry_MX_single, symbol marbastlib-mx:MX_stab
- added U1: XC6206PxxxMR, Package_TO_SOT_SMD:SOT-23-3, symbol Regulator_Linear:XC6206PxxxMR
- added U3: STM32F072C8Tx, Package_QFP:LQFP-48_7x7mm_P0.5mm, symbol MCU_ST_STM32F0:STM32F072C8Tx
- added U4: PRTR5V0U2X, Package_TO_SOT_SMD:SOT-143, symbol Power_Protection:PRTR5V0U2X
- F1: footprint Fuse:Fuse_1206_3216Metric_Pad1.42x1.75mm_HandSolder -> Fuse:Fuse_1206_3216Metric; LCSC (none) -> C135341
- R1, R2: value 22 -> 5.1k
Connections:
- net D+: now also J1.A6 (D+), J1.B6 (D+), J2.A6 (D+), J2.B6 (D+), J4.3 (Pin_3), J8.3 (Pin_3), U3.33 (PA12), U4.3 (I/O2); no longer R1.1
- net D-: now also J1.A7 (D-), J1.B7 (D-), J2.A7 (D-), J2.B7 (D-), J4.2 (Pin_2), J8.2 (Pin_2), U3.32 (PA11), U4.2 (I/O1); no longer R2.1
- net GND: now also R1.2, R2.1, C11.2, C12.2, C13.2, C14.2, C15.2, C16.2, C17.2, C18.2, C19.2, C20.2, J1.A1 (GND), J1.A12 (GND), J1.B1 (GND), J1.B12 (GND), J1.S1 (SHIELD), J2.A1 (GND), J2.A12 (GND), J2.B1 (GND), J2.B12 (GND), J2.S1 (SHIELD), J4.4 (Pin_4), J4.MP (MountPin), J8.4 (Pin_4), R10.2, RST1.2 (B), U1.1 (GND), U3.23 (VSS), U3.35 (VSS), U3.47 (VSS), U3.8 (VSSA), U4.1 (GND)
- net col0: now also K_42.1 (COL), K_64.1 (COL), K_73.1 (COL), U3.16 (PA6)
- net col1: now also K_65.1 (COL), K_68.1 (COL), K_74.1 (COL), U3.17 (PA7); no longer K_42.1 (COL)
- net col10: now also K_67.1 (COL), U3.39 (PB3)
- net col11: now also K_69.1 (COL), K_70.1 (COL), U3.40 (PB4)
- net col12: now also U3.41 (PB5)
- net col13: now also K_71.1 (COL), K_75.1 (COL), K_76.1 (COL), K_79.1 (COL), U3.42 (PB6); no longer K_41.1 (COL)
- net col14: now also K_41.1 (COL), K_72.1 (COL), K_77.1 (COL), K_78.1 (COL), K_80.1 (COL), U3.43 (PB7)
- net col2: now also U3.18 (PB0)
- net col3: now also K_66.1 (COL), U3.19 (PB1)
- net col4: now also U3.20 (PB2)
- net col5: now also U3.22 (PB11)
- net col6: now also K_62.1 (COL), K_63.1 (COL), U3.31 (PA10)
- net col7: now also U3.30 (PA9)
- net col8: now also U3.37 (PA14)
- net col9: now also U3.38 (PA15)
- net row0: now also U3.25 (PB12)
- net row1: now also U3.26 (PB13)
- net row2: now also D_64.1 (K), U3.27 (PB14)
- net row3: now also D_62.1 (K), D_63.1 (K), U3.28 (PB15)
- net row4: now also U3.29 (PA8)
- net at D_61.2 (A), K_61.2 (ROW): now also K_72.2 (ROW)
- net at D_54.2 (A), K_54.2 (ROW): now also K_64.2 (ROW)
- net at D_56.2 (A), K_56.2 (ROW): now also K_66.2 (ROW)
- net at R2.2: now also J1.B5 (CC2)
- net at D_57.2 (A), K_57.2 (ROW): now also K_62.2 (ROW), K_63.2 (ROW)
- net at D_58.2 (A), K_58.2 (ROW): now also K_67.2 (ROW)
- net at D_60.2 (A), K_60.2 (ROW): now also K_71.2 (ROW)
- net at D_59.2 (A), K_59.2 (ROW): now also K_69.2 (ROW), K_70.2 (ROW)
- net at R3.1: now also J2.A5 (CC1)
- net at D_42.2 (A): now also K_74.2 (ROW); no longer K_42.2 (ROW)
- net +5V: now reaches F1.2
- net +5V: now also C11.1, C14.1, F2.2, F4.2, U1.3 (VI), U4.4 (VCC)
- net at R4.2: now also J2.B5 (CC2)
- net at D_55.2 (A), K_55.2 (ROW): now also K_65.2 (ROW), K_68.2 (ROW)
- net at D_53.2 (A), K_53.2 (ROW): now also K_75.2 (ROW), K_76.2 (ROW)
- net at K_41.2 (ROW): now also D_64.2 (A), K_80.2 (ROW); no longer D_41.2 (A)
- net VCC: no longer names the net of F1.1
- net VCC: now also J1.A4 (VBUS), J1.A9 (VBUS), J1.B4 (VBUS), J1.B9 (VBUS)
- new net: R10.1, R9.2
- new net: F2.1, J2.A4 (VBUS), J2.A9 (VBUS), J2.B4 (VBUS), J2.B9 (VBUS)
- new net: J1.A5 (CC1), R1.1
- new net: D_41.2 (A), K_79.2 (ROW)
- new net: D_62.2 (A), K_42.2 (ROW), K_73.2 (ROW)
- new net: F4.1, J4.1 (Pin_1), J8.1 (Pin_1)
- new net: D_63.2 (A), K_77.2 (ROW), K_78.2 (ROW)
- new net +3V3: BOOT1.1 (A), C12.1, C13.1, C15.1, C16.1, C17.1, C18.1, C19.1, U1.2 (VO), U3.1 (VBAT), U3.24 (VDD), U3.36 (VDDIO2), U3.48 (VDD), U3.9 (VDDA)
- new net BOOT0: BOOT1.2 (B), R9.1, U3.44 (BOOT0)
- new net NRST: C20.1, RST1.1 (A), U3.7 (NRST)
- no-connect marks 0 -> 4
Other:
- note added: "ADC_IN8/TIM3_CH3/TTa"
- note added: "ADC_IN9/TIM3_CH4/TTa"
- note added: "DFU Mode Select (Hold while resetting to enter DFU mode)"
- note added: "Decoupling Capacitors"
- note added: "ESD, reverse polarity, and over-current protection"
- note added: "FT"
- note added: "FT/SPI1_NSS/USART2_RX"
- note added: "FT/SWCLK/USART2_TX"
- note added: "FT/SWDIO"
- note added: "FT/TIM1_CH1"
- note added: "FT/TIM1_CH2/USART1_TX"
- note added: "FT/TIM1_CH3/USART1_RX"
- note added: "I2C1_SCL/TIM16_CH1/FTf"
- note added: "I2C1_SCL/USART1_TX/FTf"
- note added: "I2C1_SDA/TIM17_CH1/FTf"
- note added: "I2C1_SDA/USART1_RX/FTf"
- note added: "I2C2_SCL/USART3_TX/TIM2_CH3/FT"
- note added: "I2C2_SDA/USART3_RX/TIM2_CH4/FT"
- note added: "NRST has internal pull-up. Capacitor holds signal stable. Optionally, remove the button, and reset by power-cycling the board."
- note added: "OSC32_IN/TC"
- note added: "OSC32_OUT/TC"
- note added: "OSC_IN/FT"
- note added: "OSC_OUT/FT"
- note added: "Power Regulation"
- note added: "Pull BOOT0 high while reseting to activate DFU."
- note added: "RESET button (Tap to reset)"
- note added: "SPI1_MISO/TIM3_CH1/FT"
- note added: "SPI1_MOSI/TIM3_CH2/FT"
- note added: "SPI1_SCK/TIM2_CH2/FT"
- note added: "SPI2_MISO/I2C2_SDA/FTf"
- note added: "SPI2_MOSI/FT"
- note added: "SPI2_NSS/FT"
- note added: "SPI2_SCK/I2C2_SCL/FTf"
- note added: "TTa/SPI1_SCK/ADC_IN5"
- note added: "TTa/TIM14_CH1/SPI1_NSS/ADC_IN4"
- note added: "TTa/TIM2_CH2/USART4_RX/ADC_IN1"
- note added: "TTa/TIM2_CH3/USART2_TX/ADC_IN2"
- note added: "TTa/TIM2_CH4/USART2_RX/ADC_IN3"
- note added: "TTa/TIM3_CH1/SPI1_MISO/ADC_IN6"
- note added: "TTa/TIM3_CH2/SPI1_MOSI/ADC_IN7"
- note added: "TTa/USART4_TX/ADC_IN0"
- note added: "WKUP2/TC"
- note added: "~10k resistor approximated with two 5.1k's from USB for BOM reduction"
- moved on the sheet: D_0, D_1, D_10, D_11, D_12, D_13, D_14, D_15, D_16, D_17, D_18, D_19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
