File: PCB/v0.3/keyboard.kicad_pcb (KiCad board)
At the start: 2 copper layers, 284.7 x 94.2 mm, 174 parts, among them J1 USB_C_Receptacle_USB2.0_16P, J2 USB_C_Receptacle_USB2.0_16P, J4 Conn_01x04_MountingPin, J8 Conn_01x04_Socket, U1 XC6206PxxxMR, U3 STM32F072C8Tx, U4 PRTR5V0U2X

Commit message: v.4
Parts:
- removed RST1: SW_SPST, Button_Switch_SMD:SW_SPST_TL3342
- added J5: Conn_01x01, TestPoint:TestPoint_Pad_3.0x3.0mm, B.Cu at (228.0, 53.5)
- added J6: Conn_01x01, TestPoint:TestPoint_Pad_3.0x3.0mm, B.Cu at (228.0, 58.8)
- added S6: MX_stab, keyboard_stabilizer:Stabilizer_Cherry_MX_2.00u, F.Cu at (257.2, -0.85)
- K_63: footprint keyboard_switches:SW_Cherry_MX_PCB_1.50u -> keyboard_switches:SW_Cherry_MX_PCB_1.25u
- moved BOOT1 86.1 mm to (155.8, 75.5), turned to 180 degrees
- moved K_63 2.38 mm to (2.38, 38.1)
Routing:
- net NRST: track 22.6 -> 154.9 mm, vias 0 -> 4
- net +3V3: track 78.2 -> 109.5 mm, vias 0 -> 2
- net BOOT0: track 47.3 -> 66.2 mm, vias 0 -> 2
- net col13: track 251.2 -> 253.6 mm
