File: PCB/v0.4/keyboard.kicad_sch (KiCad schematic)
At the start: 176 parts, among them J1 USB_C_Receptacle_USB2.0_16P, J2 USB_C_Receptacle_USB2.0_16P, J4 Conn_01x04_MountingPin, J5 Conn_01x01, J6 Conn_01x01, J8 Conn_01x04_Socket, U1 XC6206PxxxMR, U3 STM32F072C8Tx, U4 PRTR5V0U2X

Commit message: v.4
Parts:
- K_0, K_1, K_10, K_11, K_12, K_13, K_14, K_15, K_16, K_17, K_18, K_19, K_2, K_20, K_21, K_22, K_23, K_24, K_25, K_26, K_27, K_28, K_29, K_3, K_30, K_31, K_32, K_33, K_34, K_35, K_36, K_37, K_38, K_39, K_4, K_40, K_41, K_42, K_43, K_44, K_45, K_46, K_47, K_48, K_49, K_5, K_50, K_51, K_52, K_53, K_54, K_55, K_56, K_57, K_58, K_59, K_6, K_60, K_61, K_62, K_63, K_64, K_7, K_73, K_74, K_76, K_77, K_79, K_8, K_80, K_9: now not fitted
